Commit message: feat: migrate parameters to global bash environment and refactor PidController state machine to switch/case

File: src/robot_description/urdf/robot.urdf.xacro (robot description, xacro)
@@ -3,11 +3,16 @@
   <xacro:arg name="mode" default="HARDWARE"/>
   <xacro:arg name="sim_tool" default="MUJOCO"/>
-  <!-- Load hardware parameters from the global YAML -->
-  <xacro:property name="params_file" value="$(find roboteq_driver)/config/params.yaml"/>
-  <xacro:property name="hw_params" value="${xacro.load_yaml(params_file)['hardware_interface']}"/>
+  <xacro:property name="wheel_radius" value="$(optenv WHEEL_RADIUS 0.08)"/>
+  <xacro:property name="wheel_base" value="$(optenv WHEEL_BASE 0.512)"/>
+  <xacro:property name="gear_ratio" value="$(optenv GEAR_RATIO 1.0)"/>
+  <xacro:property name="ticks_per_rev" value="$(optenv TICKS_PER_REV 1024)"/>
+  <xacro:property name="left_joint_name" value="$(optenv LEFT_JOINT_NAME left_wheel_joint)"/>
+  <xacro:property name="right_joint_name" value="$(optenv RIGHT_JOINT_NAME right_wheel_joint)"/>
+  <xacro:property name="feedback_topic" value="$(optenv FEEDBACK_TOPIC /drive/feedback)"/>
+  <xacro:property name="cmd_topic" value="$(optenv CMD_TOPIC /cmd_rpm)"/>
   <!-- Minimal robot base link -->
   <link name="base_link"/>
   <!-- Left wheel joint -->
-  <joint name="${hw_params['left_joint_name']}" type="continuous">
+  <joint name="${left_joint_name}" type="continuous">
     <parent link="base_link"/>
     <child link="left_wheel"/>
@@ -16,5 +21,5 @@
   <link name="left_wheel"/>
   <!-- Right wheel joint -->
-  <joint name="${hw_params['right_joint_name']}" type="continuous">
+  <joint name="${right_joint_name}" type="continuous">
     <parent link="base_link"/>
     <child link="right_wheel"/>
@@ -27,6 +32,6 @@
       <xacro:if value="${'$(arg mode)' == 'HARDWARE'}">
         <plugin>roboteq_driver/HardwareInterface</plugin>
-        <param name="feedback_topic">${hw_params['feedback_topic']}</param>
-        <param name="cmd_topic">${hw_params['cmd_topic']}</param>
+        <param name="feedback_topic">${feedback_topic}</param>
+        <param name="cmd_topic">${cmd_topic}</param>
       </xacro:if>
       <xacro:if value="${'$(arg mode)' == 'SIM'}">
@@ -38,17 +43,17 @@
         </xacro:if>
       </xacro:if>
-      <param name="wheel_radius">${hw_params['wheel_radius']}</param>
-      <param name="wheel_base">${hw_params['wheel_base']}</param>
-      <param name="gear_ratio">${hw_params['gear_ratio']}</param>
-      <param name="ticks_per_rev">${hw_params['ticks_per_rev']}</param>
-      <param name="left_joint_name">${hw_params['left_joint_name']}</param>
-      <param name="right_joint_name">${hw_params['right_joint_name']}</param>
+      <param name="wheel_radius">${wheel_radius}</param>
+      <param name="wheel_base">${wheel_base}</param>
+      <param name="gear_ratio">${gear_ratio}</param>
+      <param name="ticks_per_rev">${ticks_per_rev}</param>
+      <param name="left_joint_name">${left_joint_name}</param>
+      <param name="right_joint_name">${right_joint_name}</param>
     </hardware>
-    <joint name="${hw_params['left_joint_name']}">
+    <joint name="${left_joint_name}">
       <command_interface name="velocity"/>
       <state_interface name="position"/>
       <state_interface name="velocity"/>
     </joint>
-    <joint name="${hw_params['right_joint_name']}">
+    <joint name="${right_joint_name}">
       <command_interface name="velocity"/>
       <state_interface name="position"/>
