Commit message: feat: path follower implementation and roboteq cross-compile fixes

File: deepak_ws/src/robot_description/urdf/robot.urdf.xacro (robot description, xacro)
@@ -13,4 +13,11 @@
   <!-- Minimal robot base link -->
   <link name="base_link"/>
+  <!-- MGS1600 Sensor Link -->
+  <joint name="mgs_sensor_joint" type="fixed">
+    <parent link="base_link"/>
+    <child link="mgs_sensor_link"/>
+    <origin xyz="0.48 0 0" rpy="0 0 0"/>
+  </joint>
+  <link name="mgs_sensor_link"/>
   <!-- Left wheel joint -->
   <joint name="${left_joint_name}" type="continuous">
